File: sheila/sheila.sch (KiCad schematic (older format))
At the start: 79 parts, among them J1 PT_A, J10 GAIN1_RETURN, J11 OT1_A, J12 OT1_B, J13 SHIELD, J14 U1A_A_1, J15 U1A_K_3, J16 TS_T, J17 TS_B, J18 TS_M, J19 TS_GND, J2 PT_B, J20 U2_K_3, J21 GAIN1_GND, J22 U1A_G_2, J23 U2_S_9, J24 U2_A_7, J25 PT_H1, J26 PT_H2, J27 LED_R, J28 LED_G, J29 LED_B, J3 PT_CT, J4 S2_A, J5 S2_B, J6 U1B_7_G, J7 U1B_6_A, J8 U1B_8_K, J9 GAIN1_SEND, Q1 BC549, U1 ECC83, U2 EL84

Commit message: Update component values
Parts:
- added J30: LED1_A, symbol Connector:Conn_01x01_Male
- J27: value LED_R -> LED1_R
- J28: value LED_G -> LED1_G
- J29: value LED_B -> LED1_B
- R5: value R_US -> 1.2K
Connections:
- net at C5.1, D3.1 (K), D4.1 (A): now also J30.1 (Pin_1)
Changed lines of the file:
@@
 P 13600 5950
 F 0 "J27" V 13650 6000 50  0000 L CNN
-F 1 "LED_R" V 13750 6000 50  0000 L CNN
+F 1 "LED1_R" V 13750 6000 50  0000 L CNN
 F 2 "" H 13600 5950 50  0001 C CNN
 F 3 "~" H 13600 5950 50  0001 C CNN
@@
 P 13350 6150
 F 0 "R5" V 13100 6150 50  0000 C CNN
-F 1 "R_US" V 13200 6150 50  0000 C CNN
+F 1 "1.2K" V 13200 6150 50  0000 C CNN
 F 2 "" V 13390 6140 50  0001 C CNN
 F 3 "~" H 13350 6150 50  0001 C CNN
@@
 P 15100 6000
 F 0 "J28" H 15050 5900 50  0000 R CNN
-F 1 "LED_G" H 15050 6000 50  0000 R CNN
+F 1 "LED1_G" H 15050 6000 50  0000 R CNN
 F 2 "" H 15100 6000 50  0001 C CNN
 F 3 "~" H 15100 6000 50  0001 C CNN
@@
 P 15100 6200
 F 0 "J29" H 15050 6100 50  0000 R CNN
-F 1 "LED_B" H 15050 6200 50  0000 R CNN
+F 1 "LED1_B" H 15050 6200 50  0000 R CNN
 F 2 "" H 15100 6200 50  0001 C CNN
 F 3 "~" H 15100 6200 50  0001 C CNN
@@
 Text Label 11050 3000 0    50   ~ 0
 A
+$Comp
+L Connector:Conn_01x01_Male J30
+U 1 1 5C5914A9
+P 14700 5350
+F 0 "J30" H 14673 5280 50  0000 R CNN
+F 1 "LED1_A" H 14673 5371 50  0000 R CNN
+F 2 "" H 14700 5350 50  0001 C CNN
+F 3 "~" H 14700 5350 50  0001 C CNN
+	1    14700 5350
+	-1   0    0    1
+$EndComp
+Connection ~ 14500 5350
 $EndSCHEMATC

Commit message: .
Parts:
- C5: value C -> 220uF/16V; footprint (none) -> Capacitor_THT:CP_Radial_D6.3mm_P2.50mm
- J25, J26, J27, J28, J29, J30: footprint (none) -> Connector_Wire:SolderWirePad_1x01_Drill0.8mm
- R11, R12, R5, R6: footprint (none) -> Resistor_THT:R_Axial_DIN0204_L3.6mm_D1.6mm_P7.62mm_Horizontal
Changed lines of the file:
@@
 U 1 1 5C6B5858
 P 13050 5800
-F 0 "C5" H 13200 5900 50  0000 L CNN
-F 1 "C" H 13200 5750 50  0000 L CNN
-F 2 "" H 13088 5650 50  0001 C CNN
+F 0 "C5" H 12900 5900 50  0000 R CNN
+F 1 "220uF/16V" H 12900 5750 50  0000 R CNN
+F 2 "Capacitor_THT:CP_Radial_D6.3mm_P2.50mm" H 13088 5650 50  0001 C CNN
 F 3 "~" H 13050 5800 50  0001 C CNN
 	1    13050 5800
@@
 F 0 "J25" H 12200 5600 50  0000 C CNN
 F 1 "PT_H1" H 12200 5500 50  0000 C CNN
-F 2 "" H 12050 5400 50  0001 C CNN
+F 2 "Connector_Wire:SolderWirePad_1x01_Drill0.8mm" H 12050 5400 50  0001 C CNN
 F 3 "~" H 12050 5400 50  0001 C CNN
 	1    12050 5400
@@
 F 0 "J26" H 12200 6000 50  0000 C CNN
 F 1 "PT_H2" H 12200 5900 50  0000 C CNN
-F 2 "" H 12050 5800 50  0001 C CNN
+F 2 "Connector_Wire:SolderWirePad_1x01_Drill0.8mm" H 12050 5800 50  0001 C CNN
 F 3 "~" H 12050 5800 50  0001 C CNN
 	1    12050 5800
@@
 F 0 "J27" V 13650 6000 50  0000 L CNN
 F 1 "LED1_R" V 13750 6000 50  0000 L CNN
-F 2 "" H 13600 5950 50  0001 C CNN
+F 2 "Connector_Wire:SolderWirePad_1x01_Drill0.8mm" H 13600 5950 50  0001 C CNN
 F 3 "~" H 13600 5950 50  0001 C CNN
 	1    13600 5950
@@
 F 0 "R5" V 13100 6150 50  0000 C CNN
 F 1 "1.2K" V 13200 6150 50  0000 C CNN
-F 2 "" V 13390 6140 50  0001 C CNN
+F 2 "Resistor_THT:R_Axial_DIN0204_L3.6mm_D1.6mm_P7.62mm_Horizontal" V 13390 6140 50  0001 C CNN
 F 3 "~" H 13350 6150 50  0001 C CNN
 	1    13350 6150
@@
 F 0 "R11" H 14400 6500 50  0000 R CNN
 F 1 "1.2K" H 14400 6350 50  0000 R CNN
-F 2 "" V 14540 6390 50  0001 C CNN
+F 2 "Resistor_THT:R_Axial_DIN0204_L3.6mm_D1.6mm_P7.62mm_Horizontal" V 14540 6390 50  0001 C CNN
 F 3 "~" H 14500 6400 50  0001 C CNN
 	1    14500 6400
@@
 F 0 "R12" H 14600 6300 50  0000 R CNN
 F 1 "1.2K" H 14600 6450 50  0000 R CNN
-F 2 "" V 14740 6390 50  0001 C CNN
+F 2 "Resistor_THT:R_Axial_DIN0204_L3.6mm_D1.6mm_P7.62mm_Horizontal" V 14740 6390 50  0001 C CNN
 F 3 "~" H 14700 6400 50  0001 C CNN
 	1    14700 6400
@@
 F 0 "R6" V 13800 6850 50  0000 C CNN
 F 1 "1M" V 13900 6850 50  0000 C CNN
-F 2 "" V 14090 6840 50  0001 C CNN
+F 2 "Resistor_THT:R_Axial_DIN0204_L3.6mm_D1.6mm_P7.62mm_Horizontal" V 14090 6840 50  0001 C CNN
 F 3 "~" H 14050 6850 50  0001 C CNN
 	1    14050 6850
@@
 F 0 "J28" H 15050 5900 50  0000 R CNN
 F 1 "LED1_G" H 15050 6000 50  0000 R CNN
-F 2 "" H 15100 6000 50  0001 C CNN
+F 2 "Connector_Wire:SolderWirePad_1x01_Drill0.8mm" H 15100 6000 50  0001 C CNN
 F 3 "~" H 15100 6000 50  0001 C CNN
 	1    15100 6000
@@
 F 0 "J29" H 15050 6100 50  0000 R CNN
 F 1 "LED1_B" H 15050 6200 50  0000 R CNN
-F 2 "" H 15100 6200 50  0001 C CNN
+F 2 "Connector_Wire:SolderWirePad_1x01_Drill0.8mm" H 15100 6200 50  0001 C CNN
 F 3 "~" H 15100 6200 50  0001 C CNN
 	1    15100 6200
@@
 F 0 "J30" H 14673 5280 50  0000 R CNN
 F 1 "LED1_A" H 14673 5371 50  0000 R CNN
-F 2 "" H 14700 5350 50  0001 C CNN
+F 2 "Connector_Wire:SolderWirePad_1x01_Drill0.8mm" H 14700 5350 50  0001 C CNN
 F 3 "~" H 14700 5350 50  0001 C CNN
 	1    14700 5350
